Commit message: update: robot's description

File: src/msds_description/urdf/msds_gazebo.xacro (robot description, xacro)
@@ -10,5 +10,5 @@
   <!-- Wheels -->
   <gazebo reference="front_right_wheel_link">
-    <material>Gazebo/Black</material>
+    <material>Gazebo/Orange</material>
     <!--
             The friction coefficient (mu1 and mu2) is a measure of the friction between the wheel and the ground.
@@ -28,5 +28,5 @@
   </gazebo>
   <gazebo reference="front_left_wheel_link">
-    <material>Gazebo/Black</material>
+    <material>Gazebo/Orange</material>
     <mu1>1000000000000000.0</mu1>
     <mu2>1000000000000000.0</mu2>

File: src/msds_description/urdf/properties.xacro (robot description, xacro)
@@ -4,10 +4,10 @@
     <xacro:property name="chassis_length" value="0.3"/>
     <xacro:property name="chassis_width" value="0.4"/>
-    <xacro:property name="chassis_height" value="0.07"/>
+    <xacro:property name="chassis_height" value="0.14"/>
     <xacro:property name="wheel_radius" value="0.0485"/>
     <xacro:property name="wheel_width" value="0.0465"/>
     <xacro:property name="lidar_height" value="0.12"/>
     <xacro:property name="imu_height" value="0.08"/>
-    <!-- Materials -->
+    <!-- Materials Colors-->
     <material name="blue">
         <color rgba="0.0 0.0 1.0 1.0"/>
@@ -24,4 +24,7 @@
     <material name="dark_grey">
         <color rgba="0.3 0.3 0.3 1"/>
+    </material>
+    <material name="orange">
+        <color rgba="0.8 0.4 0.0 1.0"/>
     </material>
     <xacro:macro name="cylinder_inertia" params="m r h xyz rpy">
