Commit message: updated robot description

File: src/msds_description/urdf/msds.urdf.xacro (robot description, xacro)
@@ -17,13 +17,26 @@
   <!-- Chassis -->
   <link name="base_link">
+    <!-- <inertial>
+      <origin xyz="0.00010187428365774479 -3.2714989699580867e-05 0.05381730231142636" rpy="0 0 0"/>
+      <mass value="8.2573504e-01"/>
+      <inertia ixx="2.2124416e-02" ixy="-1.2294101e-04" ixz="3.4938785e-04"
+            iyy="2.1193702e-02" iyz="-5.0120904e-05"
+            izz="2.0064271e-02" />
+    </inertial> -->
+    <xacro:box_inertia m="5.0" l="${2*chassis_length}" w="${2*chassis_width}" h="${2*chassis_height}"
+                           xyz="0 0 ${chassis_height / 2.0}" rpy="0 0 0"/>
     <visual>
+      <origin xyz="0 0 0" rpy="0 0 0"/>
       <geometry>
-        <box size="${chassis_length} ${chassis_width} ${chassis_height}"/>
+        <mesh filename="package://msds_description/meshes/base_link.stl" scale="0.001 0.001 0.001"/>
       </geometry>
-      <origin xyz="0 0 ${chassis_height / 2}" rpy="0 0 0"/>
-      <material name="brown">
-        <color rgba="0.6 0.4 0.2 1"/>
-      </material>
+      <material name="white"/>
     </visual>
+    <!-- <collision>
+      <origin xyz="0 0 0" rpy="0 0 0"/>
+      <geometry>
+        <mesh filename="package://msds_description/meshes/base_link.stl" scale="0.001 0.001 0.001"/>
+      </geometry>
+    </collision> -->
     <collision>
       <geometry>
@@ -32,71 +45,151 @@
       <origin xyz="0 0 ${chassis_height / 2}" rpy="0 0 0"/>
     </collision>
-    <xacro:box_inertia m="5.0" l="${2*chassis_length}" w="${2*chassis_width}" h="${2*chassis_height}"
-                           xyz="0 0 ${chassis_height / 2.0}" rpy="0 0 0"/>
   </link>
   <joint name="base_joint" type="fixed">
     <parent link="base_footprint"/>
     <child link="base_link" />
-    <origin xyz="0 0 ${wheel_radius}" rpy="0 0 0"/>
+    <origin xyz="0 0 0.081" rpy="0 0 0"/>
   </joint>
-  <!-- Wheels -->
-  <xacro:wheel name="front_left"  x="${chassis_length / 3.0}"  y="${(chassis_width + wheel_width) / 2.0}"/>
-  <xacro:wheel name="front_right" x="${chassis_length / 3.0}"  y="-${(chassis_width + wheel_width) / 2.0}"/>
-  <xacro:wheel name="rear_left"   x="-${chassis_length / 3.0}" y="${(chassis_width + wheel_width) / 2.0}"/>
-  <xacro:wheel name="rear_right"  x="-${chassis_length / 3.0}" y="-${(chassis_width + wheel_width) / 2.0}"/>
-  <!-- LIDAR -->
-  <link name="lidar_link">
+  <link name="front_right_wheel_link">
+    <xacro:cylinder_inertia m="0.152" r="${wheel_radius}" h="${wheel_width}"
+                                    xyz="0 0 0" rpy="${pi / 2.0} 0 0"/>
     <visual>
+      <origin xyz="0.2058 0.1199 0.0341" rpy="0 0 0"/>
       <geometry>
-        <cylinder radius="0.03" length="0.05"/>
+        <mesh filename="package://msds_description/meshes/front_right_link.stl" scale="0.001 0.001 0.001"/>
       </geometry>
-      <origin xyz="0 0 0" rpy="0 0 0"/>
-      <material name="black">
-        <color rgba="0.0 0.0 0.0 1.0"/>
-      </material>
+      <material name="blue"/>
     </visual>
     <collision>
       <geometry>
-        <cylinder radius="0.03" length="0.05"/>
+          <cylinder radius="${wheel_radius}" length="${wheel_width}"/>
       </geometry>
-      <origin xyz="0 0 0" rpy="0 0 0"/>
+      <origin xyz="0 0 0" rpy="${pi / 2.0} 0 0"/>
     </collision>
-    <xacro:cylinder_inertia m="0.007" r="${0.03}" h="${0.05}"
-                                    xyz="0 0 0" rpy="0 0 0"/>
   </link>
-  <joint name="lidar_joint" type="fixed">
+  <joint name="front_right_wheel_joint" type="continuous">
+    <origin xyz="-0.2058 -0.1199 -0.0341" rpy="0 0 0"/>
     <parent link="base_link"/>
-    <child link="lidar_link"/>
-    <origin xyz="0 0 ${chassis_height + 0.005}" rpy="0 0 0"/>
+    <child link="front_right_wheel_link"/>
+    <axis xyz="1 0 0" />
   </joint>
-  <!-- IMU -->
+  <link name="front_left_wheel_link">
+    <xacro:cylinder_inertia m="0.152" r="${wheel_radius}" h="${wheel_width}"
+                                    xyz="0 0 0" rpy="${pi / 2.0} 0 0"/>
+    <visual>
+      <origin xyz="-0.2058 0.1199 0.0341" rpy="0 0 0"/>
+      <geometry>
+        <mesh filename="package://msds_description/meshes/front_left_link.stl" scale="0.001 0.001 0.001"/>
+      </geometry>
+      <material name="blue"/>
+    </visual>
+    <collision>
+      <geometry>
+          <cylinder radius="${wheel_radius}" length="${wheel_width}"/>
+      </geometry>
+      <origin xyz="0 0 0" rpy="${pi / 2.0} 0 0"/>
+    </collision>
+  </link>
+  <joint name="front_left_wheel_joint" type="continuous">
+    <origin xyz="0.2058 -0.1199 -0.0341" rpy="0 0 0"/>
+    <parent link="base_link"/>
+    <child link="front_left_wheel_link"/>
+    <axis xyz="1.0 0.0 -0.0"/>
+  </joint>
+  <link name="rear_right_wheel_link">
+    <xacro:cylinder_inertia m="0.152" r="${wheel_radius}" h="${wheel_width}"
+                                    xyz="0 0 0" rpy="${pi / 2.0} 0 0"/>
+    <visual>
+      <origin xyz="0.2058 -0.1199 0.0341" rpy="0 0 0"/>
+      <geometry>
+        <mesh filename="package://msds_description/meshes/rear_right_link.stl" scale="0.001 0.001 0.001"/>
+      </geometry>
+      <material name="blue"/>
+    </visual>
+    <collision>
+      <geometry>
+          <cylinder radius="${wheel_radius}" length="${wheel_width}"/>
+      </geometry>
+      <origin xyz="0 0 0" rpy="${pi / 2.0} 0 0"/>
+    </collision>
+  </link>
+  <joint name="rear_right_wheel_joint" type="continuous">
+    <origin xyz="-0.2058 0.1199 -0.0341" rpy="0 0 0"/>
+    <parent link="base_link"/>
+    <child link="rear_right_wheel_link"/>
+    <axis xyz="-1.0 0.0 -0.0"/>
+  </joint>
+  <link name="rear_left_wheel_link">
+    <xacro:cylinder_inertia m="0.152" r="${wheel_radius}" h="${wheel_width}"
+                                    xyz="0 0 0" rpy="${pi / 2.0} 0 0"/>
+    <visual>
+      <origin xyz="-0.2058 -0.1199 0.0341" rpy="0 0 0"/>
+      <geometry>
+        <mesh filename="package://msds_description/meshes/rear_left_link.stl" scale="0.001 0.001 0.001"/>
+      </geometry>
+      <material name="blue"/>
+    </visual>
+    <collision>
+      <geometry>
+          <cylinder radius="${wheel_radius}" length="${wheel_width}"/>
+      </geometry>
+      <origin xyz="0 0 0" rpy="${pi / 2.0} 0 0"/>
+    </collision>
+  </link>
+  <joint name="rear_left_wheel_joint" type="continuous">
+    <origin xyz="0.2058 0.1199 -0.0341" rpy="0 0 0"/>
+    <parent link="base_link"/>
+    <child link="rear_left_wheel_link"/>
+    <axis xyz="-1.0 0.0 0.0"/>
+  </joint>
   <link name="imu_link">
     <inertial>
-      <origin xyz="-0.00552433659106688 0.000168210391520346 0.000514000497342681" rpy="0 0 0" />
-      <mass value="0.000528415362211671" />
-      <inertia ixx="1.46176048428261E-08" ixy="1.40015117949421E-10" ixz="-1.99633872937403E-12"
-               iyy="8.59662482954888E-09" iyz="7.52375112767959E-12"
-               izz="2.30279421279312E-08" />
+      <origin xyz="-0.020000000000000004 0.0 0.0009205607476635534" rpy="0 0 0"/>
+      <mass value="0.010079400000000002"/>
+      <inertia ixx="0.0" iyy="1e-06" izz="1e-06" ixy="-0.0" iyz="0.0" ixz="0.0"/>
     </inertial>
     <visual>
+      <origin xyz="0.107 -0.06 -0.014" rpy="0 0 0"/>
       <geometry>
-        <box size="0.03 0.03 0.01"/>
+        <mesh filename="package://msds_description/meshes/imu_link.stl" scale="0.001 0.001 0.001"/>
       </geometry>
-      <origin xyz="0.05 -0.05 0" rpy="0 0 0"/>
-      <material name="blue">
-        <color rgba="0.2 0.2 1.0 1"/>
-      </material>
+      <material name="dark_grey"/>
     </visual>
     <collision>
-      <origin xyz="0.05 -0.05 0" rpy="0 0 0"/>
+      <origin xyz="0.107 -0.06 -0.014" rpy="0 0 0"/>
       <geometry>
-        <box size="0.03 0.03 0.01"/>
+        <mesh filename="package://msds_description/meshes/imu_link.stl" scale="0.001 0.001 0.001"/>
       </geometry>
     </collision>
   </link>
   <joint name="imu_joint" type="fixed">
+    <origin xyz="-0.107 0.06 0.014" rpy="0 0 0"/>
     <parent link="base_link"/>
     <child link="imu_link"/>
-    <origin xyz="0.05 0 ${chassis_height}" rpy="0 0 0"/>
+  </joint>
+  <link name="laser_link">
+    <inertial>
+      <origin xyz="-0.049995771388990626 -0.010000165837721037 0.017999309133954644" rpy="0 0 0"/>
+      <mass value="0.7855753539396106"/>
+      <inertia ixx="0.000268" iyy="0.000268" izz="0.000331" ixy="-0.0" iyz="0.0" ixz="-0.0"/>
+    </inertial>
+    <visual>
+      <origin xyz="-0.05 0.105 -0.08" rpy="0 0 0"/>
+      <geometry>
+        <mesh filename="package://msds_description/meshes/lidar_link.stl" scale="0.001 0.001 0.001"/>
+      </geometry>
+      <material name="dark_grey"/>
+    </visual>
+    <collision>
+      <origin xyz="-0.05 0.105 -0.08" rpy="0 0 0"/>
+      <geometry>
+        <mesh filename="package://msds_description/meshes/lidar_link.stl" scale="0.001 0.001 0.001"/>
+      </geometry>
+    </collision>
+  </link>
+  <joint name="laser_joint" type="fixed">
+    <origin xyz="0.05 -0.105 0.08" rpy="0 0 0"/>
+    <parent link="base_link"/>
+    <child link="laser_link"/>
   </joint>
 </robot>

File: src/msds_description/urdf/msds_gazebo.xacro (robot description, xacro)
@@ -1,12 +1,71 @@
 <?xml version="1.0"?>
 <robot name="msds" xmlns:xacro="http://ros.org/wiki/xacro">
+  <gazebo reference="base_link">
+    <material>Gazebo/Blue</material>
+    <!-- <mu1>0.2</mu1>
+    <mu2>0.2</mu2>
+    <selfCollide>true</selfCollide>
+    <gravity>true</gravity> -->
+  </gazebo>
+  <!-- Wheels -->
+  <gazebo reference="front_right_wheel_link">
+    <material>Gazebo/Black</material>
+    <!--
+            The friction coefficient (mu1 and mu2) is a measure of the friction between the wheel and the ground.
+            A higher value indicates more friction, which can lead to better traction but also more wear on the wheels.
+            The spring constant (kp) determines how stiff the suspension is. A higher value means a stiffer suspension.
+            The damping coefficient (kd) determines how much the suspension resists motion. A higher value means more resistance.
+            The minDepth and maxVel parameters are used to limit the depth of penetration and velocity of the wheel respectively.
+            The fdir parameter specifies the direction of the friction force. It is a 3D vector that indicates the direction of the friction force.
+    -->
+    <mu1>1000000000000000.0</mu1>
+    <mu2>1000000000000000.0</mu2>
+    <kp>1000000000000.0</kp>
+    <kd>10.0</kd>
+    <minDepth>0.001</minDepth>
+    <maxVel>0.1</maxVel>
+    <fdir1>1 0 0</fdir1>
+  </gazebo>
+  <gazebo reference="front_left_wheel_link">
+    <material>Gazebo/Black</material>
+    <mu1>1000000000000000.0</mu1>
+    <mu2>1000000000000000.0</mu2>
+    <kp>1000000000000.0</kp>
+    <kd>10.0</kd>
+    <minDepth>0.001</minDepth>
+    <maxVel>0.1</maxVel>
+    <fdir1>1 0 0</fdir1>
+  </gazebo>
+  <gazebo reference="rear_right_wheel_link">
+    <material>Gazebo/Black</material>
+    <mu1>1000000000000000.0</mu1>
+    <mu2>1000000000000000.0</mu2>
+    <kp>1000000000000.0</kp>
+    <kd>10.0</kd>
+    <minDepth>0.001</minDepth>
+    <maxVel>0.1</maxVel>
+    <fdir1>1 0 0</fdir1>
+  </gazebo>
+  <gazebo reference="rear_left_wheel_link">
+    <material>Gazebo/Black</material>
+    <mu1>1000000000000000.0</mu1>
+    <mu2>1000000000000000.0</mu2>
+    <kp>1000000000000.0</kp>
+    <kd>10.0</kd>
+    <minDepth>0.001</minDepth>
+    <maxVel>0.1</maxVel>
+    <fdir1>1 0 0</fdir1>
+  </gazebo>
   <!-- ROS 2 Control -->
-  <gazebo>
+   <gazebo>
     <!-- ROS 2 Humble -->
-    <xacro:if value="$(arg is_ignition)">
+     <xacro:if value="$(arg is_ignition)">
       <plugin filename="ign_ros2_control-system" name="ign_ros2_control::IgnitionROS2ControlPlugin">
         <parameters>$(find msds_controller)/config/msds_controllers.yaml</parameters>
       </plugin>
       <plugin filename="ignition-gazebo-imu-system" name="ignition::gazebo::systems::Imu">
+      </plugin>
+      <plugin filename="ignition-gazebo-sensors-system" name="ignition::gazebo::systems::Sensors">
+        <render_engine>ogre2</render_engine>
       </plugin>
     </xacro:if>
@@ -18,4 +77,7 @@
       </plugin>
       <plugin filename="gz-sim-imu-system" name="gz::sim::systems::Imu">
+      </plugin>
+      <plugin filename="gz-sim-sensors-system" name="gz::sim::systems::Sensors">
+        <render_engine>ogre2</render_engine>
       </plugin>
     </xacro:unless>
@@ -93,28 +155,59 @@
   </gazebo>
   <!-- LIDAR -->
-  <!-- <gazebo reference="lidar_link">
-    <sensor name="lidar_sensor" type="ray">
+  <!--
+    The laser sensor is used to measure the distance to obstacles in the environment.
+    The sensor tag specifies the type of sensor and its properties.
+    The reference attribute specifies the link to which the sensor is attached - in this case, the laser_link as defined in the urdf.
+    The always_on parameter specifies whether the sensor is always on or not.
+    The update_rate parameter specifies how often the sensor readings are updated in Hz.
+    The gz_frame_id parameter specifies the frame of reference for the sensor readings.
+    The visualize parameter specifies whether the sensor is visualized in the simulation or not.
+    The topic parameter specifies the topic on which the sensor readings are published.
+    The lidar tag specifies the properties of the laser sensor.
+    The scan tag specifies the properties of the laser scan readings.
+    The horizontal tag specifies the properties of the horizontal scan readings.
+    The samples tag specifies the number of beams the laser will emit in a single scan.
+    The resolution tags specify the number of resolution of the scan.
+    The min_angle is the angle where the first beam will be emitted.
+    The max_angle is the angle where the last beam will be emitted. 360 degrees is 6.28 radians.
+    The range tag specifies the properties of the range readings.
+    The min and max tags specify how far the laser can measure.
+    The min tag is set to 0.12 meters, which means that the laser cannot measure distances closer than 0.12 meters.
+    The max tag is set to 12.0 meters, which means that the laser can measure distances up to 12.0 meters.
+    The resolution tag specifies the resolution of the range readings.
+    The noise parameters are used to simulate noise in the laser readings to make the simulation more realistic.
+    The noise type is set to gaussian, which means that the noise follows a Gaussian distribution.
+    The mean and stddev parameters specify the mean and standard deviation of the Gaussian distribution respectively.
+    The mean is set to 0.0, which means that the noise is centered around 0, and the stddev parameter specifies the standard deviation of the noise.
+    You can change some of the parameters to simulate different types of laser sensors / LIDARs.
+  -->
+  <gazebo reference="laser_link">
+    <sensor name="lidar" type="gpu_lidar">
       <always_on>true</always_on>
-      <update_rate>20.0</update_rate>
-      <ray>
+      <visualize>true</visualize>
+      <topic>scan</topic>
+      <update_rate>5</update_rate>
+      <gz_frame_id>laser_link</gz_frame_id>
+      <lidar>
         <scan>
           <horizontal>
             <samples>360</samples>
-            <resolution>1</resolution>
-            <min_angle>-3.14</min_angle>
-            <max_angle>3.14</max_angle>
+            <resolution>1.00000</resolution>
+            <min_angle>0.000000</min_angle>
+            <max_angle>6.280000</max_angle>
           </horizontal>
         </scan>
         <range>
-          <min>0.12</min>
-          <max>6.0</max>
-          <resolution>0.01</resolution>
+          <min>0.120000</min>
+          <max>12.0</max>
+          <resolution>0.02</resolution>
         </range>
-      </ray>
-      <plugin name="gazebo_ros_laser" filename="libgazebo_ros_ray_sensor.so">
-        <topicName>/scan</topicName>
-        <frameName>lidar_link</frameName>
-      </plugin>
+        <noise>
+          <type>gaussian</type>
+          <mean>0.0</mean>
+          <stddev>0.01</stddev>
+        </noise>
+      </lidar>
     </sensor>
-  </gazebo> -->
+  </gazebo>
 </robot>

File: src/msds_description/urdf/properties.xacro (robot description, xacro)
@@ -12,4 +12,16 @@
     <material name="blue">
         <color rgba="0.0 0.0 1.0 1.0"/>
+    </material>
+    <material name="black">
+        <color rgba="0 0 0 1"/>
+    </material>
+    <material name="white">
+        <color rgba="1 1 1 1"/>
+    </material>
+    <material name="silver">
+        <color rgba="0.700 0.700 0.700 1.000"/>
+    </material>
+    <material name="dark_grey">
+        <color rgba="0.3 0.3 0.3 1"/>
     </material>
     <xacro:macro name="cylinder_inertia" params="m r h xyz rpy">

Commit message: fix: laser filter problems

File: src/msds_description/urdf/msds.urdf.xacro (robot description, xacro)
@@ -170,10 +170,10 @@
   <link name="laser_link">
     <inertial>
-      <origin xyz="-0.049995771388990626 -0.010000165837721037 0.017999309133954644" rpy="0 0 0"/>
+      <origin xyz="-0.05479577138899063 -0.007200165837721026 0.017999309133954644" rpy="0 0 0"/>
       <mass value="0.7855753539396106"/>
       <inertia ixx="0.000268" iyy="0.000268" izz="0.000331" ixy="-0.0" iyz="0.0" ixz="-0.0"/>
     </inertial>
     <visual>
-      <origin xyz="-0.05 0.105 -0.08" rpy="0 0 0"/>
+      <origin xyz="-0.0 0.105 -0.08" rpy="0 0 0"/>
       <geometry>
         <mesh filename="package://msds_description/meshes/lidar_link.stl" scale="0.001 0.001 0.001"/>
@@ -189,5 +189,5 @@
   </link>
   <joint name="laser_joint" type="fixed">
-    <origin xyz="0.05 -0.105 0.08" rpy="0 0 0"/>
+    <origin xyz="0.0 -0.105 0.08" rpy="0 0 0"/>
     <parent link="base_link"/>
     <child link="laser_link"/>

Commit message: fix: bugs

File: src/msds_description/urdf/msds.urdf.xacro (robot description, xacro)
@@ -150,5 +150,5 @@
     </inertial>
     <visual>
-      <origin xyz="0.107 -0.06 -0.014" rpy="0 0 0"/>
+      <origin xyz="0.087 -0.055 -0.014" rpy="0 0 0"/>
       <geometry>
         <mesh filename="package://msds_description/meshes/imu_link.stl" scale="0.001 0.001 0.001"/>
@@ -164,5 +164,5 @@
   </link>
   <joint name="imu_joint" type="fixed">
-    <origin xyz="-0.107 0.06 0.014" rpy="0 0 0"/>
+    <origin xyz="-0.087 0.055 0.014" rpy="0 0 0"/>
     <parent link="base_link"/>
     <child link="imu_link"/>

Commit message: debugged

File: src/msds_description/urdf/msds.urdf.xacro (robot description, xacro)
@@ -49,5 +49,5 @@
     <parent link="base_footprint"/>
     <child link="base_link" />
-    <origin xyz="0 0 0.081" rpy="0 0 0"/>
+    <origin xyz="0 0 0.081" rpy="0 0 1.5708"/>
   </joint>
   <link name="front_right_wheel_link">

Commit message: fix: bugs

File: src/msds_description/urdf/msds.urdf.xacro (robot description, xacro)
@@ -49,5 +49,5 @@
     <parent link="base_footprint"/>
     <child link="base_link" />
-    <origin xyz="0 0 0.081" rpy="0 0 1.5708"/>
+    <origin xyz="0 0 0.081" rpy="0 0 ${pi / 2.0}"/>
   </joint>
   <link name="front_right_wheel_link">
@@ -189,5 +189,5 @@
   </link>
   <joint name="laser_joint" type="fixed">
-    <origin xyz="0.0 -0.105 0.08" rpy="0 0 0"/>
+    <origin xyz="0.0 -0.105 0.08" rpy="0 0 -${pi}"/>
     <parent link="base_link"/>
     <child link="laser_link"/>
